Commit message: Add gazebo features

File: arap_robot_description/urdf/mech/differential_wheel.urdf.xacro (robot description, xacro)
@@ -38,14 +38,17 @@
       <child link="${prefix}${side}_wheel_link"/>
       <origin xyz="${x_reflect*wheel_xoff} ${y_reflect*(wheel_separation/2+wheel_yoff)} ${-wheel_radius}" rpy="0 0 0"/>
+      <limit effort="30.0" velocity="10.0"/>
     </joint>
     <gazebo reference="${prefix}${side}_wheel_link">
-      <surface>
-        <friction>
-          <ode>
-              <mu>1.0</mu>
-              <mu2>0.0</mu2>
-          </ode>
-        </friction>
-      </surface>
+      <collision>
+        <surface>
+            <friction>
+                <ode>
+                    <mu>1.0</mu>
+                    <mu2>0.0</mu2>
+                </ode>
+            </friction>
+        </surface>
+      </collision>
       <visual>
           <material>
@@ -56,5 +59,5 @@
           </material>
       </visual>
-  </gazebo>
+    </gazebo>
   </xacro:macro>
 </robot>

File: arap_robot_description/urdf/sensors/imu.urdf.xacro (robot description, xacro)
@@ -64,5 +64,5 @@
                 <always_on>${always_on}</always_on>
                 <visualize>${visualize}</visualize>
-                <gz_frame_id>${prefix}${frame_id}_link</gz_frame_id>
+                <!-- <gz_frame_id>${prefix}${frame_id}_link</gz_frame_id> -->
             </sensor>
         </gazebo>

File: arap_robot_description/urdf/sensors/lidar.urdf.xacro (robot description, xacro)
@@ -105,5 +105,5 @@
           </range>
         </ray>
-        <gz_frame_id>${prefix}${frame_id}</gz_frame_id>
+        <!-- <gz_frame_id>${prefix}${frame_id}</gz_frame_id> -->
       </sensor>
     </gazebo>

File: arap_robot_description/urdf/sensors/rgbd_camera.urdf.xacro (robot description, xacro)
@@ -138,5 +138,5 @@
         </camera>
         <always_on>${always_on}</always_on>
-        <gz_frame_id>${prefix}${camera_name}_link</gz_frame_id>
+        <!-- <gz_frame_id>${prefix}${camera_name}_link</gz_frame_id> -->
         <topic>${camera_name}</topic>
         <update_rate>${update_rate}</update_rate>
