Commit message: Fix wheel rotation

File: arap_robot_description/urdf/macros/wheels.xacro (robot description, xacro)
@@ -38,6 +38,6 @@
 					<friction>
 						<ode>
-							<mu>1</mu>
-							<mu2>1</mu2>
+							<mu>10</mu>
+							<mu2>10</mu2>
 							<slip1>0.035</slip1>
 							<slip2>0</slip2>

File: arap_robot_description/urdf/robots/limo.xacro (robot description, xacro)
@@ -18,5 +18,5 @@
 	<xacro:property name="wheel_length" value="0.001" />
 	<xacro:property name="wheel_mass" value="0.5" />
-	<xacro:property name="wheel_separation" value="0.172" />
+	<xacro:property name="wheel_separation" value="0.175" />
 	<xacro:property name="max_linear_acceleration" value="1.0" />
 	<xacro:property name="kingpin_width" value="0.122" />
