Commit message: Fixed transform issues

File: arap_robot_description/urdf/macros/common.xacro (robot description, xacro)
@@ -19,5 +19,5 @@
     <!-- Output -->
     <frame_id>odom</frame_id>
-    <child_frame_id>base_link</child_frame_id>
+    <child_frame_id>base_footprint</child_frame_id>
     <odom_topic>odom</odom_topic>
     <odom_publisher_frequency>20.0</odom_publisher_frequency>

File: arap_robot_description/urdf/robots/limo.xacro (robot description, xacro)
@@ -34,13 +34,13 @@
 	<xacro:include filename="$(find arap_robot_description)/urdf/sensors/imu.xacro" />
 	<xacro:include filename="$(find arap_robot_description)/urdf/sensors/camera.xacro" />
+	<!-- BASE FOOTPRINT -->
+    <link name="base_footprint"/>
+	<joint name="base_joint" type="fixed">
+	<parent link="base_footprint"/>
+	<child link="base_link"/>
+	<origin xyz="0.0 0.0 0.0" rpy="0 0 0"/>
+	</joint>
 	<!-- Base link -->
 	<link name="base_link"/>
-	<!-- BASE FOOTPRINT -->
-    <link name="base_footprint"/>
-    <joint name="base_joint" type="fixed">
-        <parent link="base_link"/>
-        <child link="base_footprint"/>
-        <origin xyz="0.0 0.0 0.0" rpy="0 0 0"/>
-    </joint>
 	<!-- Chassis -->
 	<joint name="chassis_joint" type="fixed">
