Commit message: Added Nav2 configurations

File: arap_robot_description/urdf/control/diff/gazebo_control.xacro (robot description, xacro)
@@ -15,4 +15,5 @@
 		</plugin>
 		<xacro:joint_state_publisher_plugin />
+		<xacro:pose_publisher_plugin />
 	</gazebo>
 </robot>

File: arap_robot_description/urdf/macros/common.xacro (robot description, xacro)
@@ -1,45 +1,60 @@
 <?xml version="1.0"?>
 <robot xmlns:xacro="http://www.ros.org/wiki/xacro">
-	<!-- Joint State Publisher Plugin -->
-	<xacro:macro name="joint_state_publisher_plugin">
-		<plugin filename="gz-sim-joint-state-publisher-system"
-			name="gz::sim::systems::JointStatePublisher">
-			<topic>joint_states</topic>
-			<joint_name>front_left_wheel_joint</joint_name>
-			<joint_name>front_right_wheel_joint</joint_name>
-			<joint_name>rear_left_wheel_joint</joint_name>
-			<joint_name>rear_right_wheel_joint</joint_name>
-		</plugin>
-	</xacro:macro>
-	<!-- Common Gazebo Control Plugin Parameters -->
-	<xacro:macro name="gazebo_control_common_plugin_params">
-		<!-- Input -->
-		<topic>cmd_vel</topic>
-		<!-- Output -->
-		<frame_id>odom</frame_id>
-		<child_frame_id>base_link</child_frame_id>
-		<odom_topic>odom</odom_topic>
-		<odom_publisher_frequency>30</odom_publisher_frequency>
-		<tf_topic>/tf</tf_topic>
-	</xacro:macro>
-	<xacro:macro name="wheel_setup" params="wheel_type config">
-		<xacro:property name="wheel_type" value="${wheel_type}" />
-		<!-- Wheels -->
-		<xacro:wheel wheel_prefix="front_left" parent_prefix="base_link" reflect="1"
-			wheel_type="${wheel_type}">
-			<origin xyz="${wheelbase/2} ${track/2} ${wheel_vertical_offset}" rpy="0 0 0" />
-		</xacro:wheel>
-		<xacro:wheel wheel_prefix="front_right" parent_prefix="base_link" reflect="-1"
-			wheel_type="${wheel_type}">
-			<origin xyz="${wheelbase/2} ${-track/2} ${wheel_vertical_offset}" rpy="${M_PI} 0 0" />
-		</xacro:wheel>
-		<xacro:wheel wheel_prefix="rear_left" parent_prefix="base_link" reflect="1"
-			wheel_type="${wheel_type}">
-			<origin xyz="${-wheelbase/2} ${track/2} ${wheel_vertical_offset}" rpy="0 0 0" />
-		</xacro:wheel>
-		<xacro:wheel wheel_prefix="rear_right" parent_prefix="base_link" reflect="-1"
-			wheel_type="${wheel_type}">
-			<origin xyz="${-wheelbase/2} ${-track/2} ${wheel_vertical_offset}" rpy="${M_PI} 0 0" />
-		</xacro:wheel>
-	</xacro:macro>
+  <!-- Joint State Publisher Plugin -->
+  <xacro:macro name="joint_state_publisher_plugin">
+    <plugin filename="gz-sim-joint-state-publisher-system"
+      name="gz::sim::systems::JointStatePublisher">
+      <topic>joint_states</topic>
+      <joint_name>front_left_wheel_joint</joint_name>
+      <joint_name>front_right_wheel_joint</joint_name>
+      <joint_name>rear_left_wheel_joint</joint_name>
+      <joint_name>rear_right_wheel_joint</joint_name>
+    </plugin>
+  </xacro:macro>
+  <!-- Common Gazebo Control Plugin Parameters -->
+  <xacro:macro name="gazebo_control_common_plugin_params">
+    <!-- Input -->
+    <topic>cmd_vel</topic>
+    <!-- Output -->
+    <frame_id>odom</frame_id>
+    <child_frame_id>base_link</child_frame_id>
+    <odom_topic>odom</odom_topic>
+    <odom_publisher_frequency>30</odom_publisher_frequency>
+    <tf_topic>/tf</tf_topic>
+    <publish_odom_tf>true</publish_odom_tf>
+    <publish_wheel_tf>true</publish_wheel_tf>
+    <odometry_source>world</odometry_source>
+    <update_rate>30.0</update_rate>
+  </xacro:macro>
+  <xacro:macro name="wheel_setup" params="wheel_type config">
+    <xacro:property name="wheel_type" value="${wheel_type}" />
+    <!-- Wheels -->
+    <xacro:wheel wheel_prefix="front_left" parent_prefix="base_link" reflect="1"
+      wheel_type="${wheel_type}">
+      <origin xyz="${wheelbase/2} ${track/2} ${wheel_vertical_offset}" rpy="0 0 0" />
+    </xacro:wheel>
+    <xacro:wheel wheel_prefix="front_right" parent_prefix="base_link" reflect="-1"
+      wheel_type="${wheel_type}">
+      <origin xyz="${wheelbase/2} ${-track/2} ${wheel_vertical_offset}" rpy="${M_PI} 0 0" />
+    </xacro:wheel>
+    <xacro:wheel wheel_prefix="rear_left" parent_prefix="base_link" reflect="1"
+      wheel_type="${wheel_type}">
+      <origin xyz="${-wheelbase/2} ${track/2} ${wheel_vertical_offset}" rpy="0 0 0" />
+    </xacro:wheel>
+    <xacro:wheel wheel_prefix="rear_right" parent_prefix="base_link" reflect="-1"
+      wheel_type="${wheel_type}">
+      <origin xyz="${-wheelbase/2} ${-track/2} ${wheel_vertical_offset}" rpy="${M_PI} 0 0" />
+    </xacro:wheel>
+  </xacro:macro>
+  <!-- Pose Publisher Plugin Macro -->
+  <xacro:macro name="pose_publisher_plugin">
+    <plugin filename="gz-sim-pose-publisher-system" name="gz::sim::systems::PosePublisher">
+      <publish_link_pose>true</publish_link_pose>
+      <publish_collision_pose>false</publish_collision_pose>
+      <publish_visual_pose>false</publish_visual_pose>
+      <publish_nested_model_pose>false</publish_nested_model_pose>
+      <use_pose_vector_msg>true</use_pose_vector_msg>
+      <update_rate>30.0</update_rate>
+    </plugin>
+  </xacro:macro>
 </robot>

File: arap_robot_description/urdf/sensors/imu.xacro (robot description, xacro)
@@ -34,4 +34,5 @@
                 <always_on>true</always_on>
                 <update_rate>100</update_rate>
+                <frame_name>imu_link</frame_name>
                 <visualize>true</visualize>
                 <imu>

File: arap_robot_description/urdf/sensors/laser.xacro (robot description, xacro)
@@ -56,4 +56,5 @@
 				</lidar>
 				<topic>scan</topic>
+				<frame_name>laser_frame</frame_name>
 				<gz_frame_id>laser_frame</gz_frame_id>
 			</sensor>

Commit message: Add steer spinning to robot description

File: arap_robot_description/urdf/control/diff/gazebo_control.xacro (robot description, xacro)
@@ -3,14 +3,16 @@
 	<gazebo>
 		<plugin name="gz::sim::systems::DiffDrive" filename="gz-sim-diff-drive-system">
-			<!-- Wheel Information -->
-			<!-- <left_joint>front_left_wheel_joint</left_joint>
-			<right_joint>front_right_wheel_joint</right_joint> -->
-			<left_joint>rear_left_wheel_joint</left_joint>
-			<right_joint>rear_right_wheel_joint</right_joint>
-			<wheel_separation>${wheel_separation}</wheel_separation>
-			<wheel_radius>${wheel_radius}</wheel_radius>
-			<!-- Limits -->
-			<max_linear_acceleration>${max_linear_acceleration}</max_linear_acceleration>
-			<xacro:gazebo_control_common_plugin_params />
+		<!-- Wheel Information -->
+		<left_joint>front_left_wheel_joint</left_joint>
+		<left_joint>rear_left_wheel_joint</left_joint>
+		<right_joint>front_right_wheel_joint</right_joint>
+		<right_joint>rear_right_wheel_joint</right_joint>
+		<wheel_separation>${wheel_separation}</wheel_separation>
+		<wheel_radius>${wheel_radius}</wheel_radius>
+		<!-- Additional control parameters -->
+		<max_linear_acceleration>${max_linear_acceleration}</max_linear_acceleration>
+  		<max_angular_acceleration>2.0</max_angular_acceleration>
+		<skid_steering>true</skid_steering>
+		<xacro:gazebo_control_common_plugin_params />
 		</plugin>
 		<xacro:joint_state_publisher_plugin />

File: arap_robot_description/urdf/macros/common.xacro (robot description, xacro)
@@ -10,4 +10,5 @@
       <joint_name>rear_left_wheel_joint</joint_name>
       <joint_name>rear_right_wheel_joint</joint_name>
+      <update_rate>20</update_rate>
     </plugin>
   </xacro:macro>
@@ -20,10 +21,10 @@
     <child_frame_id>base_link</child_frame_id>
     <odom_topic>odom</odom_topic>
-    <odom_publisher_frequency>30</odom_publisher_frequency>
+    <odom_publisher_frequency>20.0</odom_publisher_frequency>
     <tf_topic>/tf</tf_topic>
     <publish_odom_tf>true</publish_odom_tf>
-    <publish_wheel_tf>true</publish_wheel_tf>
+    <publish_wheel_tf>false</publish_wheel_tf>
     <odometry_source>world</odometry_source>
-    <update_rate>30.0</update_rate>
+    <update_rate>20.0</update_rate>
   </xacro:macro>
   <xacro:macro name="wheel_setup" params="wheel_type config">
@@ -55,5 +56,5 @@
       <publish_nested_model_pose>false</publish_nested_model_pose>
       <use_pose_vector_msg>true</use_pose_vector_msg>
-      <update_rate>30.0</update_rate>
+      <update_rate>20.0</update_rate>
     </plugin>
   </xacro:macro>

File: arap_robot_description/urdf/macros/wheels.xacro (robot description, xacro)
@@ -38,10 +38,15 @@
 					<friction>
 						<ode>
-							<mu>10</mu>
-							<mu2>10</mu2>
-							<slip1>0.035</slip1>
-							<slip2>0</slip2>
+							<mu>1.0</mu>
+							<mu2>0.5</mu2>
+							<slip1>0.001</slip1>
+							<slip2>0.001</slip2>
 							<fdir1>0 0 1</fdir1>
 						</ode>
+						<bullet>
+							<friction>1</friction>
+							<friction2>1</friction2>
+							<rolling_friction>0.1</rolling_friction>
+						</bullet>
 					</friction>
 				</surface>

File: arap_robot_description/urdf/robots/limo.xacro (robot description, xacro)
@@ -15,8 +15,8 @@
 	<xacro:property name="track" value="0.13" />
 	<xacro:property name="wheel_vertical_offset" value="0.05" />
-	<xacro:property name="wheel_radius" value="0.045" />
+	<xacro:property name="wheel_radius" value="0.0325" />
 	<xacro:property name="wheel_length" value="0.001" />
 	<xacro:property name="wheel_mass" value="0.5" />
-	<xacro:property name="wheel_separation" value="0.175" />
+	<xacro:property name="wheel_separation" value="0.170" />
 	<xacro:property name="max_linear_acceleration" value="1.0" />
 	<xacro:property name="kingpin_width" value="0.122" />
@@ -32,4 +32,11 @@
 	<!-- Base link -->
 	<link name="base_link" />
+	    <!-- BASE FOOTPRINT -->
+    <link name="base_footprint"/>
+    <joint name="base_footprint_joint" type="fixed">
+        <parent link="base_link"/>
+        <child link="base_footprint"/>
+        <origin xyz="0 0 0" rpy="0 0 0"/>
+    </joint>
 	<!-- Chassis -->
 	<joint name="chassis_joint" type="fixed">

Commit message: Fix synchronization issue between ROS and Gazebo

File: arap_robot_description/urdf/control/diff/gazebo_control.xacro (robot description, xacro)
@@ -3,4 +3,6 @@
 	<gazebo>
 		<plugin name="gz::sim::systems::DiffDrive" filename="gz-sim-diff-drive-system">
+		<update_rate>100</update_rate>
+		<num_wheel_pairs>2</num_wheel_pairs>
 		<!-- Wheel Information -->
 		<left_joint>front_left_wheel_joint</left_joint>
@@ -8,10 +10,19 @@
 		<right_joint>front_right_wheel_joint</right_joint>
 		<right_joint>rear_right_wheel_joint</right_joint>
-		<wheel_separation>${wheel_separation}</wheel_separation>
-		<wheel_radius>${wheel_radius}</wheel_radius>
-		<!-- Additional control parameters -->
-		<max_linear_acceleration>${max_linear_acceleration}</max_linear_acceleration>
-  		<max_angular_acceleration>2.0</max_angular_acceleration>
-		<skid_steering>true</skid_steering>
+		<wheel_separation>0.172</wheel_separation>
+		<!-- <wheel_radius>${wheel_radius}</wheel_radius> -->
+		<wheel_radius>0.0225</wheel_radius> <!-- Wheel Diameter = 0.09; Wheel Radius = 0.045 -->
+		<!-- Limits -->
+		<max_wheel_torque>100</max_wheel_torque>
+		<max_wheel_acceleration>5.0</max_wheel_acceleration>
+		<command_topic>cmd_vel</command_topic> <!-- Fully qualified topics begin with '/' -->
+		<publish_odom>true</publish_odom>
+		<publish_odom_tf>true</publish_odom_tf>
+		<publish_wheel_tf>true</publish_wheel_tf>
+		<odometry_topic>odom</odometry_topic>
+		<odometry_frame>odom</odometry_frame>
+		<robot_base_frame>base_footprint</robot_base_frame>
+		<odometry_source>1</odometry_source>
+		<skid_steering>false</skid_steering>
 		<xacro:gazebo_control_common_plugin_params />
 		</plugin>

File: arap_robot_description/urdf/macros/common.xacro (robot description, xacro)
@@ -26,5 +26,5 @@
     <publish_wheel_tf>false</publish_wheel_tf>
     <odometry_source>world</odometry_source>
-    <update_rate>20.0</update_rate>
+    <update_rate>100.0</update_rate>
   </xacro:macro>
   <xacro:macro name="wheel_setup" params="wheel_type config">

File: arap_robot_description/urdf/macros/wheels.xacro (robot description, xacro)
@@ -9,5 +9,5 @@
 			<axis xyz="0 ${reflect*1} 0">
 				<limit>
-					<effort>20</effort>
+					<effort>100</effort>
 				</limit>
 			</axis>
@@ -39,14 +39,11 @@
 						<ode>
 							<mu>1.0</mu>
-							<mu2>0.5</mu2>
-							<slip1>0.001</slip1>
-							<slip2>0.001</slip2>
-							<fdir1>0 0 1</fdir1>
+							<mu2>1.0</mu2>
+							<kp>100.0</kp>
+							<kd>1.0</kd>
+							<minDepth>0.01</minDepth>
+							<fdir1>1 0 0</fdir1>
+							<maxContacts value="64" />
 						</ode>
-						<bullet>
-							<friction>1</friction>
-							<friction2>1</friction2>
-							<rolling_friction>0.1</rolling_friction>
-						</bullet>
 					</friction>
 				</surface>

File: arap_robot_description/urdf/robots/limo.xacro (robot description, xacro)
@@ -12,11 +12,15 @@
 	<!-- Robot Variables -->
 	<xacro:property name="base_mass" value="2.1557" />
+	<!-- Robot Geometries -->
+	<xacro:property name="base_x_size" value="0.13" />
+	<xacro:property name="base_y_size" value="0.12" />
+	<xacro:property name="base_z_size" value="0.1" />
 	<xacro:property name="wheelbase" value="0.2" />
 	<xacro:property name="track" value="0.13" />
 	<xacro:property name="wheel_vertical_offset" value="0.05" />
-	<xacro:property name="wheel_radius" value="0.0325" />
-	<xacro:property name="wheel_length" value="0.001" />
-	<xacro:property name="wheel_mass" value="0.5" />
-	<xacro:property name="wheel_separation" value="0.170" />
+	<xacro:property name="wheel_radius" value="0.0225" /> <!-- Possible values: (0.0325 / 2), 0.048, 0.042, 0.01625 -->
+	<xacro:property name="wheel_length" value="0.045" />
+	<xacro:property name="wheel_mass" value="0.5" /> <!-- Initially 0.5 -->
+	<xacro:property name="wheel_separation" value="0.13" /> <!-- Initially 0.170 (Calculates the distance between the two wheels - on the y-axis) -->
 	<xacro:property name="max_linear_acceleration" value="1.0" />
 	<xacro:property name="kingpin_width" value="0.122" />
@@ -31,17 +35,17 @@
 	<xacro:include filename="$(find arap_robot_description)/urdf/sensors/camera.xacro" />
 	<!-- Base link -->
-	<link name="base_link" />
-	    <!-- BASE FOOTPRINT -->
+	<link name="base_link"/>
+	<!-- BASE FOOTPRINT -->
     <link name="base_footprint"/>
-    <joint name="base_footprint_joint" type="fixed">
+    <joint name="base_joint" type="fixed">
         <parent link="base_link"/>
         <child link="base_footprint"/>
-        <origin xyz="0 0 0" rpy="0 0 0"/>
+        <origin xyz="0.0 0.0 0.0" rpy="0 0 0"/>
     </joint>
 	<!-- Chassis -->
 	<joint name="chassis_joint" type="fixed">
-		<parent link="base_link" />
-		<child link="chassis" />
-		<origin xyz="0.0 0.0 0.15" />
+		<parent link="base_link"/>
+		<child link="chassis"/>
+		<origin xyz="0.0 0.0 0.15"/>
 	</joint>
 	<link name="chassis">
@@ -56,6 +60,5 @@
 			<origin xyz="0 0 -0.15" rpy="0 0 1.57" />
 			<geometry>
-				<mesh filename="package://arap_robot_description/meshes/chassis/chassis.stl"
-					scale="1 1 1" />
+				<mesh filename="package://arap_robot_description/meshes/chassis/chassis.stl" scale="1 1 1" />
 			</geometry>
 		</collision>
@@ -72,5 +75,5 @@
 	</xacro:laser>
 	<xacro:camera parent_prefix="chassis">
-		<origin xyz="0.084 0 0.026" rpy="0 0 0" />
+		<origin xyz="0.084 0 0.03" rpy="0 0 0" />
 	</xacro:camera>
 	<xacro:imu parent_prefix="chassis">

File: arap_robot_description/urdf/sensors/imu.xacro (robot description, xacro)
@@ -31,4 +31,5 @@
         </joint>
         <gazebo reference="imu_link">
+            <gravity>true</gravity>
             <sensor name="imu" type="imu">
                 <always_on>true</always_on>
@@ -37,4 +38,24 @@
                 <visualize>true</visualize>
                 <imu>
+                    <orientation>
+                        <x>
+                            <noise type="gaussian">
+                                <mean>0.0</mean>
+                                <stddev>2e-3</stddev>
+                            </noise>
+                        </x>
+                        <y>
+                            <noise type="gaussian">
+                                <mean>0.0</mean>
+                                <stddev>2e-3</stddev>
+                            </noise>
+                        </y>
+                        <z>
+                            <noise type="gaussian">
+                                <mean>0.0</mean>
+                                <stddev>2e-3</stddev>
+                            </noise>
+                        </z>
+                    </orientation>
                     <angular_velocity>
                         <x>

File: arap_robot_description/urdf/sensors/laser.xacro (robot description, xacro)
@@ -34,18 +34,18 @@
 				<always_on>true</always_on>
 				<visualize>true</visualize>
-				<update_rate>2</update_rate>
+				<update_rate>10</update_rate>
 				<lidar>
 					<scan>
 						<horizontal>
-							<samples>720</samples>
-							<resolution>1</resolution>
-							<min_angle>-2.09439504</min_angle>
-							<max_angle>2.09439504</max_angle>
+							<samples>120</samples>
+							<resolution>1.000000</resolution>
+							<min_angle>-3.14159</min_angle>
+							<max_angle>3.14159</max_angle>
 						</horizontal>
 					</scan>
 					<range>
-						<min>0.05</min>
-						<max>8.0</max>
-						<resolution>0.01</resolution>
+						<min>0.3</min>
+						<max>15.0</max>
+						<resolution>0.015</resolution>
 					</range>
 					<noise>
